File: kicad/solderbit-gamepad.kicad_sch (KiCad schematic)
At the start: 34 parts, among them J1 Microbit_Edge_Connector, J2 S2B-PH-SM4-TB(LF)(SN), Q1 DMG2045U, SW1 MST22D18G2 125, U1 74HC165D,653, U2 NCP114ASN330T1G

Commit message: Replace all with v0.9 and new media
Parts:
- removed C3, C4, C5, C6: 1uF, Solderbit_Gamepad:1206_Capacitor, symbol Solderbit_Gamepad:Capacitor
- removed J1: Microbit_Edge_Connector, Solderbit_Gamepad:Microbit_Edge_Connector, symbol Solderbit_Gamepad:Microbit_Edge_Connector
- removed R2, R3, R4, R5, R6, R8: 100k, Solderbit_Gamepad:1206_Resistor, symbol Solderbit_Gamepad:Resistor
- removed S8: TS-1037-A4B3-D2, Solderbit_Gamepad:Tactile_Switch_Right_90_Degrees, symbol Solderbit_Gamepad:Tactile_Switch_2_Pin
- added CN1, CN2, CN3, CN4, CN5: SMTSOM310BTR, Solderbit_Gamepad:SMTSOM310BTR, symbol Virtual_Modules:SMTSO4020MTJ
- BT1: Basic No -> (none); Part type (none) -> Extended; now left out of the parts list
- C1, C2, C7, C8, R1, R7, R9: Basic Yes -> (none); Part type (none) -> Basic
- D1, D6, J2, R10, S1, S7, SW1: Basic No -> (none); Part type (none) -> Extended
- H1, H2, H3, H4: now left out of the parts list
- Q1, U2: Part type (none) -> Extended
- U1: Basic No -> (none); Package SOIC-16 -> SOIC-16; Part type (none) -> Extended promotional
Connections:
- net CLK: now also CN3.1
- net GND: now also CN5.1
- net PL/DATA: now also CN2.1
- net SER: now also CN1.1
- net Vubit: now also CN4.1
Other:
- note added: "100k resistor"
- note added: "1uF capacitor"
- note added: "3V"
- note added: "GND"
- note added: "P1"
- note added: "P2"
- note added: "PO"
- note added: "WS2812B"
- note added: "hint"
- note added: "micro:bit SMTSO adaptor"
- note added: "tact switch"
- note added: "tact switch 90-degrees"
- note removed: "micro:bit edge connector"
- company: pro² network+ summer school 2025 -> Devices Lab & pro² network+
- moved on the sheet: C2, D1, R7, R9, S7

Commit message: Cleanup, and add new images
Connections:
- no-connect marks 5 -> 6
